File: Drone_PCB/Drone_PCB.kicad_sch (KiCad schematic)
At the start: 44 parts, among them J1 Conn_01x04_Pin, J2 Conn_01x04_Pin, J3 Conn_01x04_Pin, J4 Conn_01x06_Pin, J5 Conn_01x06_Pin, J6 USB_B_Micro, Q1 BSS214NW, Q2 BSS214NW, SW2 SW_DPST_x2, U1 STM32F411RCT6, U2 AP2112K-3.3, U3 TP4056-42-ESOP8, U4 DW01A, Y1 26MHz

Commit message: Creating PCB part 1
Circuit is looking pretty neat
Parts:
- removed Y1: 26MHz, Crystal:Crystal_SMD_HC49-SD, symbol Device:Crystal_GND24
- added Y1: 26MHz, Crystal:Crystal_SMD_HC49-SD, symbol Device:Crystal
Connections:
- net HSE_IN: now also Y1.1
- net HSE_OUT: now also Y1.2
Changed lines of the file:
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@@
 	)
 	(junction
-		(at 171.45 82.55)
-		(diameter 0)
-		(color 0 0 0 0)
-	)
-	(junction
 		(at 60.96 110.49)
 		(diameter 0)
@@
 	)
 	(junction
-		(at 171.45 87.63)
-		(diameter 0)
-		(color 0 0 0 0)
-	)
-	(junction
 		(at 39.37 45.72)
 		(diameter 0)
@@
 	)
 	(junction
-		(at 148.59 39.37)
+		(at 181.61 78.74)
 		(diameter 0)
 		(color 0 0 0 0)
 	)
 	(junction
-		(at 45.72 185.42)
+		(at 148.59 39.37)
 		(diameter 0)
 		(color 0 0 0 0)
 	)
 	(junction
-		(at 157.48 76.2)
+		(at 45.72 185.42)
 		(diameter 0)
 		(color 0 0 0 0)
@@
 	)
 	(junction
+		(at 157.48 78.74)
+		(diameter 0)
+		(color 0 0 0 0)
+	)
+	(junction
 		(at 137.16 49.53)
 		(diameter 0)
@@
 	)
 	(junction
-		(at 181.61 76.2)
-		(diameter 0)
-		(color 0 0 0 0)
-	)
-	(junction
 		(at 236.22 49.53)
 		(diameter 0)
@@
 	(wire
 		(pts
-			(xy 181.61 76.2) (xy 181.61 78.74)
+			(xy 181.61 71.12) (xy 181.61 78.74)
 		)
 		(stroke
@@
 	(wire
 		(pts
-			(xy 166.37 69.85) (xy 166.37 82.55)
-		)
-		(stroke
-			(width 0)
-			(type default)
-		)
-	)
-	(wire
-		(pts
 			(xy 137.16 39.37) (xy 148.59 39.37)
 		)
@@
 	(wire
 		(pts
-			(xy 166.37 82.55) (xy 171.45 82.55)
-		)
-		(stroke
-			(width 0)
-			(type default)
-		)
-	)
-	(wire
-		(pts
 			(xy 254 76.2) (xy 251.46 76.2)
 		)
@@
 	(wire
 		(pts
-			(xy 157.48 76.2) (xy 157.48 78.74)
-		)
-		(stroke
-			(width 0)
-			(type default)
-		)
-	)
-	(wire
-		(pts
 			(xy 73.66 44.45) (xy 73.66 45.72)
 		)
@@
 	(wire
 		(pts
-			(xy 171.45 69.85) (xy 166.37 69.85)
-		)
-		(stroke
-			(width 0)
-			(type default)
-		)
-	)
-	(wire
-		(pts
 			(xy 167.64 120.65) (xy 179.07 120.65)
 		)
@@
 	(wire
 		(pts
-			(xy 157.48 87.63) (xy 171.45 87.63)
-		)
-		(stroke
-			(width 0)
-			(type default)
-		)
-	)
-	(wire
-		(pts
 			(xy 236.22 49.53) (xy 236.22 50.8)
 		)
@@
 	(wire
 		(pts
-			(xy 157.48 68.58) (xy 157.48 76.2)
+			(xy 157.48 68.58) (xy 157.48 78.74)
 		)
 		(stroke
@@
 	(wire
 		(pts
-			(xy 171.45 87.63) (xy 181.61 87.63)
+			(xy 157.48 87.63) (xy 181.61 87.63)
 		)
 		(stroke
@@
 	(wire
 		(pts
-			(xy 171.45 71.12) (xy 171.45 69.85)
-		)
-		(stroke
-			(width 0)
-			(type default)
-		)
-	)
-	(wire
-		(pts
 			(xy 19.05 57.15) (xy 39.37 57.15)
 		)
@@
 	(wire
 		(pts
-			(xy 181.61 71.12) (xy 181.61 76.2)
-		)
-		(stroke
-			(width 0)
-			(type default)
-		)
-	)
-	(wire
-		(pts
 			(xy 167.64 96.52) (xy 191.77 96.52)
 		)
@@
 	(wire
 		(pts
-			(xy 181.61 76.2) (xy 175.26 76.2)
-		)
-		(stroke
-			(width 0)
-			(type default)
-		)
-	)
-	(wire
-		(pts
 			(xy 57.15 57.15) (xy 73.66 57.15)
 		)
@@
 	(wire
 		(pts
-			(xy 171.45 82.55) (xy 171.45 87.63)
-		)
-		(stroke
-			(width 0)
-			(type default)
-		)
-	)
-	(wire
-		(pts
 			(xy 207.01 49.53) (xy 209.55 49.53)
 		)
@@
 	(wire
 		(pts
+			(xy 175.26 78.74) (xy 181.61 78.74)
+		)
+		(stroke
+			(width 0)
+			(type default)
+		)
+	)
+	(wire
+		(pts
 			(xy 73.66 54.61) (xy 73.66 57.15)
 		)
@@
 	(wire
 		(pts
+			(xy 157.48 78.74) (xy 167.64 78.74)
+		)
+		(stroke
+			(width 0)
+			(type default)
+		)
+	)
+	(wire
+		(pts
 			(xy 60.96 152.4) (xy 82.55 152.4)
 		)
@@
 	(wire
 		(pts
-			(xy 167.64 76.2) (xy 157.48 76.2)
-		)
-		(stroke
-			(width 0)
-			(type default)
-		)
-	)
-	(wire
-		(pts
 			(xy 167.64 99.06) (xy 191.77 99.06)
 		)
@@
 	(wire
 		(pts
-			(xy 171.45 81.28) (xy 171.45 82.55)
-		)
-		(stroke
-			(width 0)
-			(type default)
-		)
-	)
-	(wire
-		(pts
 			(xy 154.94 67.31) (xy 154.94 68.58)
 		)
@@
 	)
 	(symbol
+		(lib_id "Device:Crystal")
+		(at 171.45 78.74 0)
+		(unit 1)
+		(exclude_from_sim no)
+		(in_bom yes)
+		(on_board yes)
+		(dnp no)
+		(fields_autoplaced yes)
+		(property "Reference" "Y1"
+			(at 171.45 71.12 0)
+			(effects
+				(font
+					(size 1.27 1.27)
+				)
+			)
+		)
+		(property "Value" "26MHz"
+			(at 171.45 73.66 0)
+			(effects
+				(font
+					(size 1.27 1.27)
+				)
+			)
+		)
+		(property "Footprint" "Crystal:Crystal_SMD_HC49-SD"
+			(at 171.45 78.74 0)
+			(effects
+				(font
+					(size 1.27 1.27)
+				)
+				(hide yes)
+			)
+		)
+		(property "Datasheet" "~"
+			(at 171.45 78.74 0)
+			(effects
+				(font
+					(size 1.27 1.27)
+				)
+				(hide yes)
+			)
+		)
+		(property "Description" "Two pin crystal"
+			(at 171.45 78.74 0)
+			(effects
+				(font
+					(size 1.27 1.27)
+				)
+				(hide yes)
+			)
+		)
+		(pin "2"
+		)
+		(pin "1"
+		)
+		(instances
+			(project ""
+				(path "/2c198202-91eb-4035-8605-360d42f3c3f5"
+					(reference "Y1")
+					(unit 1)
+				)
+			)
+		)
+	)
+	(symbol
 		(lib_id "Device:C")
 		(at 90.17 152.4 90)
@@
 					(unit 1)
 				)
-			)
-		)
-	)
-	(symbol
-		(lib_id "Device:Crystal_GND24")
-		(at 171.45 76.2 0)
-		(unit 1)
-		(exclude_from_sim no)
-		(in_bom yes)
-		(on_board yes)
-		(dnp no)
-		(property "Reference" "Y1"
-			(at 175.514 72.898 0)
-			(effects
-				(font
-					(size 1.27 1.27)
-				)
-			)
-		)
-		(property "Value" "26MHz"
-			(at 177.546 78.232 0)
-			(effects
-				(font
-					(size 1.27 1.27)
-				)
-			)
-		)
-		(property "Footprint" "Crystal:Crystal_SMD_HC49-SD"
-			(at 171.45 76.2 0)
-			(effects
-				(font
-					(size 1.27 1.27)
-				)
-				(hide yes)
-			)
-		)
-		(property "Datasheet" "~"
-			(at 171.45 76.2 0)
-			(effects
-				(font
-					(size 1.27 1.27)
-				)
-				(hide yes)
-			)
-		)
-		(property "Description" "Four pin crystal, GND on pins 2 and 4"
-			(at 171.45 76.2 0)
-			(effects
-				(font
-					(size 1.27 1.27)
-				)
-				(hide yes)
-			)
-		)
-		(pin "4"
-		)
-		(pin "1"
-		)
-		(pin "2"
-		)
-		(pin "3"
-		)
-		(instances
-			(project ""
-				(path "/2c198202-91eb-4035-8605-360d42f3c3f5"
-					(reference "Y1")
-					(unit 1)
-				)
